File: PcbTUT.kicad_pcb (KiCad board)
At the start: 2 copper layers, 77.1 x 38.1 mm, 24 parts, among them SW1 SW_Push, U1 ATmega32U4-AU, Y1 16Mhz

Commit message: Finalized v.01
Parts:
- moved USB1 0.15 mm to (72.6, 81.1)
Routing:
- net Net-(USB1-Pad6): track 0.00 -> 16.3 mm
- net COL0: track 35.5 -> 36.4 mm
- added copper zone on B.Cu, net (none)
- added copper zone on F.Cu, net (none)
- added copper zone on B.Cu, net GND
Other:
- board text added: "NetClicker V.01"
- board text added: "SpikedSynapse"
Changed lines of the file:
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@@
   (general
     (thickness 1.6)
-    (drawings 8)
-    (tracks 186)
+    (drawings 10)
+    (tracks 190)
     (zones 0)
     (modules 24)
@@
     (pcbplotparams
       (layerselection 0x010fc_ffffffff)
-      (usegerberextensions false)
+      (usegerberextensions true)
       (usegerberattributes true)
       (usegerberadvancedattributes true)
-      (creategerberjobfile true)
+      (creategerberjobfile false)
       (excludeedgelayer true)
-      (linewidth 0.100000)
+      (linewidth 0.020000)
       (plotframeref false)
       (viasonmask false)
@@
       (plotinvisibletext false)
       (padsonsilk false)
-      (subtractmaskfromsilk false)
+      (subtractmaskfromsilk true)
       (outputformat 1)
       (mirror false)
-      (drillshape 1)
+      (drillshape 0)
       (scaleselection 1)
-      (outputdirectory ""))
+      (outputdirectory "Gerbers/"))
   )
   (net 0 "")
@@
   )
   (module random-keyboard-parts:Molex-0548190589 (layer B.Cu)
-    (at 72.644 81.28 270)
+    (at 72.644 81.1276 270)
     (attr smd)
     (fp_text reference USB1 (at 2.032 0) (layer B.SilkS)
@@
       (rotate (xyz 0 0 0))
     )
+  )
+  (gr_text "NetClicker V.01" (at 86.36 115.316) (layer F.SilkS)
+    (effects (font (size 0.508 0.508) (thickness 0.0508)))
+  )
+  (gr_text SpikedSynapse (at 86.36 114.3) (layer F.Mask)
+    (effects (font (size 0.762 0.762) (thickness 0.15)))
   )
   (gr_line (start 64.16675 115.09375) (end 64.516 81.788) (layer Edge.Cuts) (width 0.05))
@@
   (segment (start 108.9025 86.36) (end 108.9025 105.41) (width 0.254) (layer F.Cu) (net 12))
   (segment (start 108.9025 105.41) (end 108.9025 104.8385) (width 0.254) (layer F.Cu) (net 12))
-  (segment (start 101.6 100.076) (end 95.2985 100.076) (width 0.254) (layer B.Cu) (net 12))
+  (segment (start 106.934 105.41) (end 108.9025 105.41) (width 0.254) (layer B.Cu) (net 12))
+  (segment (start 103.064038 101.540038) (end 106.934 105.41) (width 0.254) (layer B.Cu) (net 12))
   (segment (start 95.2985 100.076) (end 95.235 100.1395) (width 0.254) (layer B.Cu) (net 12))
-  (segment (start 108.9025 105.41) (end 106.934 105.41) (width 0.254) (layer B.Cu) (net 12))
-  (segment (start 106.934 105.41) (end 101.6 100.076) (width 0.254) (layer B.Cu) (net 12))
+  (segment (start 103.064038 100.076) (end 95.2985 100.076) (width 0.254) (layer B.Cu) (net 12))
+  (segment (start 103.064038 101.540038) (end 103.064038 100.076) (width 0.254) (layer B.Cu) (net 12))
   (segment (start 127.9525 86.36) (end 127.9525 105.41) (width 0.254) (layer F.Cu) (net 13))
   (segment (start 127.6985 105.156) (end 127.9525 105.41) (width 0.254) (layer B.Cu) (net 13))
@@
   (segment (start 87.884 91.899632) (end 88.735 92.750632) (width 0.254) (layer B.Cu) (net 41))
   (segment (start 87.884 89.408) (end 87.884 91.899632) (width 0.254) (layer B.Cu) (net 41))
+  (segment (start 76.294 85.6276) (end 76.294 81.1276) (width 0.254) (layer B.Cu) (net 44))
+  (segment (start 76.294 81.1276) (end 68.994 81.1276) (width 0.254) (layer B.Cu) (net 44))
+  (segment (start 68.994 81.1276) (end 68.994 85.6276) (width 0.254) (layer B.Cu) (net 44))
+  (zone (net 1) (net_name GND) (layer B.Cu) (hatch edge 0.508)
+    (connect_pads (clearance 0.508))
+    (min_thickness 0.254)
+    (fill yes (arc_segments 32) (thermal_gap 0.508) (thermal_bridge_width 0.508))
+    (polygon
+      (pts
+        (xy 95.504 106.68) (xy 83.82 106.68) (xy 83.82 93.98) (xy 95.504 93.98)
+      )
+    )
+  )
+  (zone (net 1) (net_name GND) (layer B.Cu) (hatch edge 0.508)
+    (connect_pads (clearance 0.508))
+    (min_thickness 0.254)
+    (fill yes (arc_segments 32) (thermal_gap 0.508) (thermal_bridge_width 0.508))
+    (polygon
+      (pts
+        (xy 98.044 86.36) (xy 98.044 89.916) (xy 96.52 91.44) (xy 83.312 91.44) (xy 81.28 89.408)
+        (xy 81.28 86.36) (xy 82.804 84.836) (xy 96.52 84.836)
+      )
+    )
+  )
+  (zone (net 0) (net_name "") (layer B.Cu) (hatch edge 0.508)
+    (connect_pads (clearance 0.508))
+    (min_thickness 0.254)
+    (fill yes (arc_segments 32) (thermal_gap 0.508) (thermal_bridge_width 0.508))
+    (polygon
+      (pts
+        (xy 91.44 113.792) (xy 91.44 115.316) (xy 90.424 116.332) (xy 82.296 116.332) (xy 81.28 115.316)
+        (xy 81.28 113.792) (xy 82.296 112.776) (xy 90.424 112.776)
+      )
+    )
+  )
+  (zone (net 0) (net_name "") (layer F.Cu) (hatch edge 0.508)
+    (connect_pads (clearance 0.508))
+    (min_thickness 0.254)
+    (fill yes (arc_segments 32) (thermal_gap 0.508) (thermal_bridge_width 0.508))
+    (polygon
+      (pts
+        (xy 91.44 113.284) (xy 91.44 115.824) (xy 90.932 116.332) (xy 81.788 116.332) (xy 81.28 115.824)
+        (xy 81.28 113.284) (xy 81.788 112.776) (xy 90.932 112.776)
+      )
+    )
+  )
+  (zone (net 1) (net_name GND) (layer B.Cu) (hatch edge 0.508)
+    (connect_pads (clearance 0.508))
+    (min_thickness 0.254)
+    (fill yes (arc_segments 32) (thermal_gap 0.508) (thermal_bridge_width 0.508))
+    (polygon
+      (pts
+        (xy 78.2828 80.1624) (xy 78.2828 87.0204) (xy 67.2084 86.9188) (xy 67.31 80.0608)
+      )
+    )
+  )
 )
